File: hardware/Jopen-backups/Jopen.kicad_sch (KiCad schematic)
At the start: 21 parts, among them J6 Screw_Terminal_01x18, J7 Screw_Terminal_01x18, U2 TPS7B6933QDCYRQ1

Commit message: Fix P1 IN3 and P2 ADC4 pin configuration
Firmware changes:
- Disabled ADC peripheral initialization (MX_ADC1_Init and HAL_ADC_MspInit)
- Added GPIO pull-up resistors for all button inputs (active-low logic)
- Fixed keyboard HID descriptor (6KRO standard format, 47 bytes)
- Added LED debug indicators (LED1=P1, LED2=P2)
- Device name now conditional based on mode (Keyboard/Joystick/JVS)
- Fixed pin mappings for dual arcade controls (34 inputs total)

Hardware changes:
- Updated KiCad files (v6+ format)
- Added netlist (Jopen.net) for pin verification
- Added flash.ps1 script for automated programming
Connections:
- net GND: now also D1.1 (K); no longer D1.2 (K)
- net at R35.1: now also D1.2 (A); no longer D1.1 (A)
- net +3V3 renamed +3.3V
