File: hardware/Jopen-backups/mcu.kicad_sch (KiCad schematic)
At the start: 121 parts, among them U1 STM32F102RBTx, Y1 8 MHz

Commit message: Fix P1 IN3 and P2 ADC4 pin configuration
Firmware changes:
- Disabled ADC peripheral initialization (MX_ADC1_Init and HAL_ADC_MspInit)
- Added GPIO pull-up resistors for all button inputs (active-low logic)
- Fixed keyboard HID descriptor (6KRO standard format, 47 bytes)
- Added LED debug indicators (LED1=P1, LED2=P2)
- Device name now conditional based on mode (Keyboard/Joystick/JVS)
- Fixed pin mappings for dual arcade controls (34 inputs total)

Hardware changes:
- Updated KiCad files (v6+ format)
- Added netlist (Jopen.net) for pin verification
- Added flash.ps1 script for automated programming
Connections:
- net GND: now also D2.1 (K), D3.1 (K), D4.1 (K); no longer D2.2 (K), D3.2 (K), D4.2 (K)
- net LED1: no longer U1.51 (PC10)
- net LED2: no longer U1.52 (PC11)
- net LED3: no longer U1.53 (PC12)
- net OSC_IN: now also U1.25 (PC5); no longer U1.5 (PD0)
- net OSC_OUT: now also U1.37 (PC6); no longer U1.6 (PD1)
- net uC_ADC1: now also U1.53 (PC12); no longer U1.11 (PC3)
- net uC_ADC2: now also U1.52 (PC11); no longer U1.10 (PC2)
- net uC_IN1: now also U1.51 (PC10); no longer U1.9 (PC1)
- net uC_IN14: now also U1.2 (PC13); no longer U1.24 (PC4)
- net uC_IN15: now also U1.3 (PC14); no longer U1.25 (PC5)
- net uC_IN2: now also U1.40 (PC9); no longer U1.8 (PC0)
- net uC_IN23: no longer U1.39 (PC8)
- net uC_IN24: no longer U1.40 (PC9)
- net uC_IN3: no longer U1.4 (PC15)
- net uC_IN4: no longer U1.3 (PC14)
- net uC_IN5: no longer U1.2 (PC13)
- net uC_TIM3: now also U1.4 (PC15); no longer U1.37 (PC6)
- net uC_TIM4: no longer U1.38 (PC7)
- net at R1.2: now also U1.38 (PC7); no longer U1.54 (PD2)
- net at R41.2: now also D4.2 (A); no longer D4.1 (A)
- net at R40.2: now also D3.2 (A); no longer D3.1 (A)
- net at R39.2: now also D2.2 (A); no longer D2.1 (A)
- net +3V3 renamed +3.3V
